File: ltc3440.sch (KiCad schematic (older format))
At the start: 9 parts, among them U1 LTC3440EDD

Commit message: layout board
Parts:
- added J1: Conn_01x04, Connector_PinSocket_2.54mm:PinSocket_1x04_P2.54mm_Vertical, symbol Connector_Generic:Conn_01x04
Connections:
- net +3V3: now also J1.1 (Pin_1)
- net +BATT: now also J1.3 (Pin_3)
- net GND: now also J1.2 (Pin_2), J1.4 (Pin_4)
Changed lines of the file:
@@
 Wire Wire Line
 	5300 2950 4900 2950
-$Comp
-L power:+BATT #PWR01
-U 1 1 5F6C24BC
-P 4450 2800
-F 0 "#PWR01" H 4450 2650 50  0001 C CNN
-F 1 "+BATT" H 4465 2973 50  0000 C CNN
-F 2 "" H 4450 2800 50  0001 C CNN
-F 3 "" H 4450 2800 50  0001 C CNN
-	1    4450 2800
-	1    0    0    -1
-$EndComp
 Wire Wire Line
 	4450 2800 4450 2950
@@
 Fixed Freq. Mode
 $Comp
-L power:PWR_FLAG #FLG?
+L power:PWR_FLAG #FLG0101
 U 1 1 5F742A39
 P 4900 2950
-F 0 "#FLG?" H 4900 3025 50  0001 C CNN
+F 0 "#FLG0101" H 4900 3025 50  0001 C CNN
 F 1 "PWR_FLAG" H 4900 3123 50  0000 C CNN
 F 2 "" H 4900 2950 50  0001 C CNN
@@
 $EndComp
 $Comp
-L power:PWR_FLAG #FLG?
+L power:PWR_FLAG #FLG0102
 U 1 1 5F743DCE
 P 6800 3000
-F 0 "#FLG?" H 6800 3075 50  0001 C CNN
+F 0 "#FLG0102" H 6800 3075 50  0001 C CNN
 F 1 "PWR_FLAG" H 6800 3173 50  0000 C CNN
 F 2 "" H 6800 3000 50  0001 C CNN
@@
 $EndComp
 $Comp
-L power:PWR_FLAG #FLG?
+L power:PWR_FLAG #FLG0103
 U 1 1 5F74412F
 P 6800 4300
-F 0 "#FLG?" H 6800 4375 50  0001 C CNN
+F 0 "#FLG0103" H 6800 4375 50  0001 C CNN
 F 1 "PWR_FLAG" H 6800 4473 50  0000 C CNN
 F 2 "" H 6800 4300 50  0001 C CNN
@@
 	-1   0    0    1
 $EndComp
+$Comp
+L power:+BATT #PWR01
+U 1 1 5F6C24BC
+P 4450 2800
+F 0 "#PWR01" H 4450 2650 50  0001 C CNN
+F 1 "+BATT" H 4465 2973 50  0000 C CNN
+F 2 "" H 4450 2800 50  0001 C CNN
+F 3 "" H 4450 2800 50  0001 C CNN
+	1    4450 2800
+	1    0    0    -1
+$EndComp
+$Comp
+L Connector_Generic:Conn_01x04 J1
+U 1 1 5F76521E
+P 8600 3000
+F 0 "J1" H 8680 2992 50  0000 L CNN
+F 1 "Conn_01x04" H 8680 2901 50  0000 L CNN
+F 2 "Connector_PinSocket_2.54mm:PinSocket_1x04_P2.54mm_Vertical" H 8600 3000 50  0001 C CNN
+F 3 "~" H 8600 3000 50  0001 C CNN
+	1    8600 3000
+	1    0    0    -1
+$EndComp
+$Comp
+L power:+3.3V #PWR0101
+U 1 1 5F766D52
+P 8300 2800
+F 0 "#PWR0101" H 8300 2650 50  0001 C CNN
+F 1 "+3.3V" H 8315 2973 50  0000 C CNN
+F 2 "" H 8300 2800 50  0001 C CNN
+F 3 "" H 8300 2800 50  0001 C CNN
+	1    8300 2800
+	1    0    0    -1
+$EndComp
+$Comp
+L power:+BATT #PWR0102
+U 1 1 5F767E3D
+P 8000 2800
+F 0 "#PWR0102" H 8000 2650 50  0001 C CNN
+F 1 "+BATT" H 8015 2973 50  0000 C CNN
+F 2 "" H 8000 2800 50  0001 C CNN
+F 3 "" H 8000 2800 50  0001 C CNN
+	1    8000 2800
+	1    0    0    -1
+$EndComp
+Wire Wire Line
+	8300 2800 8300 2900
+Wire Wire Line
+	8300 2900 8400 2900
+Wire Wire Line
+	8000 3100 8400 3100
+Wire Wire Line
+	8000 2800 8000 3100
+$Comp
+L power:GND #PWR0103
+U 1 1 5F76AAC7
+P 8300 3350
+F 0 "#PWR0103" H 8300 3100 50  0001 C CNN
+F 1 "GND" H 8305 3177 50  0000 C CNN
+F 2 "" H 8300 3350 50  0001 C CNN
+F 3 "" H 8300 3350 50  0001 C CNN
+	1    8300 3350
+	1    0    0    -1
+$EndComp
+Wire Wire Line
+	8400 3000 8300 3000
+Wire Wire Line
+	8300 3000 8300 3200
+Wire Wire Line
+	8400 3200 8300 3200
+Connection ~ 8300 3200
+Wire Wire Line
+	8300 3200 8300 3350
 $EndSCHEMATC

Commit message: change to burst mode
Connections:
- net +BATT: now also U1.2 (MODE/SYNC)
- net GND: no longer U1.2 (MODE/SYNC)
Other:
- note added: "Burst Mode"
- note removed: "Fixed Freq. Mode"
Changed lines of the file:
@@
 Wire Wire Line
 	4600 4200 4600 4300
-Wire Wire Line
-	4600 4300 4900 4300
 Connection ~ 5500 4300
 Wire Wire Line
@@
 	5000 3700 4900 3700
 Wire Wire Line
-	4900 3700 4900 4300
-Connection ~ 4900 4300
-Wire Wire Line
-	4900 4300 5500 4300
-Wire Wire Line
 	4450 2950 4450 3500
-Wire Wire Line
-	5000 3500 4900 3500
-Wire Wire Line
-	4900 3500 4900 2950
 Connection ~ 4900 2950
 Wire Wire Line
@@
 VOUT voltage set by R1,R2 on FB\nVOUT = 1.22* (1+R1/R2)
 Connection ~ 6400 3000
-$Comp
-L Device:R_Small RT1
-U 1 1 5F6B5037
-P 4600 4100
-F 0 "RT1" H 4659 4146 50  0000 L CNN
-F 1 "60.4k" H 4659 4055 50  0000 L CNN
-F 2 "Resistor_SMD:R_0603_1608Metric_Pad1.05x0.95mm_HandSolder" H 4600 4100 50  0001 C CNN
-F 3 "~" H 4600 4100 50  0001 C CNN
-	1    4600 4100
-	1    0    0    -1
-$EndComp
 $Comp
 L ltc3440:LTC3440EDD U1
@@
 Wire Wire Line
 	6800 3000 7150 3000
-Text Notes 4450 4400 0    50   ~ 0
-Fixed Freq. Mode
 $Comp
 L power:PWR_FLAG #FLG0101
@@
 Wire Wire Line
 	8300 3200 8300 3350
+Text Notes 4630 3800 0    50   ~ 0
+Burst Mode
+$Comp
+L Device:R_Small RT1
+U 1 1 5F6B5037
+P 4600 4100
+F 0 "RT1" H 4659 4146 50  0000 L CNN
+F 1 "60.4k" H 4659 4055 50  0000 L CNN
+F 2 "Resistor_SMD:R_0603_1608Metric_Pad1.05x0.95mm_HandSolder" H 4600 4100 50  0001 C CNN
+F 3 "~" H 4600 4100 50  0001 C CNN
+	1    4600 4100
+	1    0    0    -1
+$EndComp
+Wire Wire Line
+	5000 3500 4900 3500
+Wire Wire Line
+	4600 4300 5500 4300
+Wire Wire Line
+	4900 2950 4900 3500
+Connection ~ 4900 3500
+Wire Wire Line
+	4900 3500 4900 3700
 $EndSCHEMATC

Commit message: change inductor with smaller footprint
Parts:
- L1: footprint ltc3440:L_Sumida-CDRH6D38 -> ltc3440:IND_LQH5BPN100M38L; Digikey_PN 308-1541-2-ND -> 490-16631-1-ND; MPN CDRH6D38-100 -> LQH5BPN100M38L; Manufacturer SUMIDA -> Murata Electronics
Changed lines of the file:
@@
 F 0 "L1" V 5967 2950 50  0000 C CNN
 F 1 "10uH" V 5876 2950 50  0000 C CNN
-F 2 "ltc3440:L_Sumida-CDRH6D38" H 5600 2950 50  0001 C CNN
+F 2 "ltc3440:IND_LQH5BPN100M38L" H 5600 2950 50  0001 C CNN
 F 3 "~" H 5600 2950 50  0001 C CNN
-F 4 "CDRH6D38-100" V 5785 2950 50  0000 C CNN "MPN"
-F 5 "SUMIDA " V 5694 2950 50  0000 C CNN "Manufacturer"
-F 6 "308-1541-2-ND" V 5600 2950 50  0001 C CNN "Digikey_PN"
+F 4 "LQH5BPN100M38L" V 5785 2950 50  0000 C CNN "MPN"
+F 5 "Murata Electronics" V 5694 2950 50  0000 C CNN "Manufacturer"
+F 6 "490-16631-1-ND" V 5600 2950 50  0001 C CNN "Digikey_PN"
 	1    5600 2950
 	0    -1   -1   0

Commit message: fix error sw2 to vout
Connections:
- net +3V3: no longer L1.2, U1.4 (SW2)
- new net: L1.2, U1.4 (SW2)
Changed lines of the file:
@@
 $EndComp
-Wire Wire Line
-	5700 2950 5700 3000
 Wire Wire Line
 	5500 4200 5500 4300
@@
 Wire Wire Line
 	6100 3300 6400 3300
-Wire Wire Line
-	6400 3000 5700 3000
-Connection ~ 5700 3000
-Wire Wire Line
-	5700 3000 5700 3100
 Wire Wire Line
 	6400 3000 6800 3000
@@
 Text Notes 6200 4750 0    50   ~ 0
 VOUT voltage set by R1,R2 on FB\nVOUT = 1.22* (1+R1/R2)
-Connection ~ 6400 3000
 $Comp
 L ltc3440:LTC3440EDD U1
@@
 Wire Wire Line
 	4900 3500 4900 3700
+Wire Wire Line
+	5700 2950 5700 3100
 $EndSCHEMATC
